Commit message: Updated with TCP links

File: gateway_description/robots/big_arm.urdf.xacro (robot description, xacro)
@@ -6,3 +6,9 @@
     <origin xyz="0.0 0.0 0.0" rpy="0.0 0.4363 -1.396"/>
   </xacro:big_arm>
+  <link name="big_arm_link_tcp"/>
+  <joint name="big_arm_tcp_joint" type="fixed">
+    <parent link="big_arm_link_8"/>
+    <child link="big_arm_link_tcp"/>
+    <origin xyz="0 0 0" rpy="0 0 0"/>
+  </joint>
 </robot>

File: gateway_description/robots/little_arm.urdf.xacro (robot description, xacro)
@@ -6,3 +6,9 @@
     <origin xyz="0.0 0.0 0.0" rpy="0.0 0.4363 -1.396"/>
   </xacro:little_arm>
+  <link name="little_arm_link_tcp"/>
+  <joint name="little_arm_tcp" type="fixed">
+    <parent link="little_arm_link_8"/>
+    <child link="little_arm_link_tcp"/>
+    <origin xyz="0 0 0" rpy="0 0 0"/>
+  </joint>
 </robot>
