Commit message: Updated with  ros1 changes to make robots more modular

File: gateway_description/robots/original_urdf/gateway_original.urdf.xacro (robot description, xacro)
@@ -192,15 +192,15 @@
     </collision>
   </link>
-  <joint name="joint_big_arm_joint_0" type="fixed">
+  <joint name="big_arm_joint_0" type="fixed">
     <parent link="root"/>
     <child link="big_arm_link_0"/>
     <origin xyz="0.0 0.0 0.0" rpy="0.0 0.4363 -1.396"/>
   </joint>
-  <joint name="joint_big_arm_joint_1" type="fixed">
+  <joint name="big_arm_joint_1" type="fixed">
     <parent link="big_arm_link_0"/>
     <child link="big_arm_link_1"/>
     <origin xyz="3.7698 0.3139 1.6058" rpy="0.0 -0.2094 -1.5708"/>
   </joint>
-  <joint name="joint_big_arm_joint_2" type="revolute">
+  <joint name="big_arm_joint_2" type="revolute">
     <parent link="big_arm_link_1"/>
     <child link="big_arm_link_2"/>
@@ -209,5 +209,5 @@
     <origin xyz="0.0 0.0 0.4409" rpy="0.0 0.0 0.8726648"/>
   </joint>
-  <joint name="joint_big_arm_joint_3" type="revolute">
+  <joint name="big_arm_joint_3" type="revolute">
     <parent link="big_arm_link_2"/>
     <child link="big_arm_link_3"/>
@@ -216,5 +216,5 @@
     <limit lower="-1.5708" upper="1.5708" velocity="100" effort="100"/> <!-- MADE UP NUMBERS JUST FOR TESTING -->
   </joint>
-  <joint name="joint_big_arm_joint_4" type="revolute">
+  <joint name="big_arm_joint_4" type="revolute">
     <parent link="big_arm_link_3"/>
     <child link="big_arm_link_4"/>
@@ -223,5 +223,5 @@
     <limit lower="-1.5708" upper="1.5708" velocity="100" effort="100"/> <!-- MADE UP NUMBERS JUST FOR TESTING -->
   </joint>
-  <joint name="joint_big_arm_joint_5" type="revolute">
+  <joint name="big_arm_joint_5" type="revolute">
     <parent link="big_arm_link_4"/>
     <child link="big_arm_link_5"/>
@@ -230,5 +230,5 @@
     <limit lower="-1.5708" upper="1.5708" velocity="100" effort="100"/> <!-- MADE UP NUMBERS JUST FOR TESTING -->
   </joint>
-  <joint name="joint_big_arm_joint_6" type="revolute">
+  <joint name="big_arm_joint_6" type="revolute">
     <parent link="big_arm_link_5"/>
     <child link="big_arm_link_6"/>
@@ -237,5 +237,5 @@
     <limit lower="-1.5708" upper="1.5708" velocity="100" effort="100"/> <!-- MADE UP NUMBERS JUST FOR TESTING -->
   </joint>
-  <joint name="joint_big_arm_joint_7" type="revolute">
+  <joint name="big_arm_joint_7" type="revolute">
     <parent link="big_arm_link_6"/>
     <child link="big_arm_link_7"/>
@@ -244,5 +244,5 @@
     <limit lower="-1.5708" upper="1.5708" velocity="100" effort="100"/> <!-- MADE UP NUMBERS JUST FOR TESTING -->
   </joint>
-  <joint name="joint_big_arm_joint_8" type="revolute">
+  <joint name="big_arm_joint_8" type="revolute">
     <parent link="big_arm_link_7"/>
     <child link="big_arm_link_8"/>
@@ -361,15 +361,15 @@
     </collision>
   </link>
-  <joint name="joint_little_arm_joint_0" type="fixed">
+  <joint name="little_arm_joint_0" type="fixed">
     <parent link="root"/>
     <child link="little_arm_link_0"/>
     <origin xyz="0.0 0.0 0.0" rpy="0.0 0.4363 -1.396"/>
   </joint>
-  <joint name="joint_little_arm_joint_1" type="fixed">
+  <joint name="little_arm_joint_1" type="fixed">
     <parent link="little_arm_link_0"/>
     <child link="little_arm_link_1"/>
     <origin xyz="13.984 -1.3352 -1.3367" rpy="2.3562 0.0 0.0"/>
   </joint>
-  <joint name="joint_little_arm_joint_2" type="revolute">
+  <joint name="little_arm_joint_2" type="revolute">
     <parent link="little_arm_link_1"/>
     <child link="little_arm_link_2"/>
@@ -378,5 +378,5 @@
     <origin xyz="0.44043 0.010424 0.29487" rpy="0.0 0.0 0.0"/>
   </joint>
-  <joint name="joint_little_arm_joint_3" type="revolute">
+  <joint name="little_arm_joint_3" type="revolute">
     <parent link="little_arm_link_2"/>
     <child link="little_arm_link_3"/>
@@ -385,5 +385,5 @@
     <limit lower="-1.5708" upper="1.5708" velocity="100" effort="100"/> <!-- MADE UP NUMBERS JUST FOR TESTING -->
   </joint>
-  <joint name="joint_little_arm_joint_4" type="revolute">
+  <joint name="little_arm_joint_4" type="revolute">
     <parent link="little_arm_link_3"/>
     <child link="little_arm_link_4"/>
@@ -392,5 +392,5 @@
     <limit lower="-1.5708" upper="1.5708" velocity="100" effort="100"/> <!-- MADE UP NUMBERS JUST FOR TESTING -->
   </joint>
-  <joint name="joint_little_arm_joint_5" type="revolute">
+  <joint name="little_arm_joint_5" type="revolute">
     <parent link="little_arm_link_4"/>
     <child link="little_arm_link_5"/>
@@ -399,5 +399,5 @@
     <limit lower="-1.5708" upper="1.5708" velocity="100" effort="100"/> <!-- MADE UP NUMBERS JUST FOR TESTING -->
   </joint>
-  <joint name="joint_little_arm_joint_6" type="revolute">
+  <joint name="little_arm_joint_6" type="revolute">
     <parent link="little_arm_link_5"/>
     <child link="little_arm_link_6"/>
@@ -406,5 +406,5 @@
     <limit lower="-1.5708" upper="1.5708" velocity="100" effort="100"/> <!-- MADE UP NUMBERS JUST FOR TESTING -->
   </joint>
-  <joint name="joint_little_arm_joint_7" type="revolute">
+  <joint name="little_arm_joint_7" type="revolute">
     <parent link="little_arm_link_6"/>
     <child link="little_arm_link_7"/>
@@ -413,5 +413,5 @@
     <limit lower="-1.5708" upper="1.5708" velocity="100" effort="100"/> <!-- MADE UP NUMBERS JUST FOR TESTING -->
   </joint>
-  <joint name="joint_little_arm_joint_8" type="revolute">
+  <joint name="little_arm_joint_8" type="revolute">
     <parent link="little_arm_link_7"/>
     <child link="little_arm_link_8"/>
@@ -420,5 +420,5 @@
     <limit lower="-1.5708" upper="1.5708" velocity="100" effort="100"/> <!-- MADE UP NUMBERS JUST FOR TESTING -->
   </joint>
-  <joint name="joint_little_arm_joint_9" type="revolute">
+  <joint name="little_arm_joint_9" type="revolute">
     <parent link="little_arm_link_8"/>
     <child link="little_arm_link_9"/>

File: gateway_description/xacro/big_arm_macro.xacro (robot description, xacro)
@@ -100,15 +100,15 @@
     </collision>
   </link>
-  <joint name="joint_big_arm_joint_0" type="fixed">
+  <joint name="big_arm_joint_0" type="fixed">
     <parent link="${parent}"/>
     <child link="big_arm_link_0"/>
     <xacro:insert_block name="origin"/>
   </joint>
-  <joint name="joint_big_arm_joint_1" type="fixed">
+  <joint name="big_arm_joint_1" type="fixed">
     <parent link="big_arm_link_0"/>
     <child link="big_arm_link_1"/>
     <origin xyz="3.7698 0.3139 1.6058" rpy="0.0 -0.2094 -1.5708"/>
   </joint>
-  <joint name="joint_big_arm_joint_2" type="revolute">
+  <joint name="big_arm_joint_2" type="revolute">
     <parent link="big_arm_link_1"/>
     <child link="big_arm_link_2"/>
@@ -117,5 +117,5 @@
     <origin xyz="0.0 0.0 0.4409" rpy="0.0 0.0 0.8726648"/>
   </joint>
-  <joint name="joint_big_arm_joint_3" type="revolute">
+  <joint name="big_arm_joint_3" type="revolute">
     <parent link="big_arm_link_2"/>
     <child link="big_arm_link_3"/>
@@ -124,5 +124,5 @@
     <limit lower="-1.5708" upper="1.5708" velocity="100" effort="100"/> <!-- MADE UP NUMBERS JUST FOR TESTING -->
   </joint>
-  <joint name="joint_big_arm_joint_4" type="revolute">
+  <joint name="big_arm_joint_4" type="revolute">
     <parent link="big_arm_link_3"/>
     <child link="big_arm_link_4"/>
@@ -131,5 +131,5 @@
     <limit lower="-1.5708" upper="1.5708" velocity="100" effort="100"/> <!-- MADE UP NUMBERS JUST FOR TESTING -->
   </joint>
-  <joint name="joint_big_arm_joint_5" type="revolute">
+  <joint name="big_arm_joint_5" type="revolute">
     <parent link="big_arm_link_4"/>
     <child link="big_arm_link_5"/>
@@ -138,5 +138,5 @@
     <limit lower="-1.5708" upper="1.5708" velocity="100" effort="100"/> <!-- MADE UP NUMBERS JUST FOR TESTING -->
   </joint>
-  <joint name="joint_big_arm_joint_6" type="revolute">
+  <joint name="big_arm_joint_6" type="revolute">
     <parent link="big_arm_link_5"/>
     <child link="big_arm_link_6"/>
@@ -145,5 +145,5 @@
     <limit lower="-1.5708" upper="1.5708" velocity="100" effort="100"/> <!-- MADE UP NUMBERS JUST FOR TESTING -->
   </joint>
-  <joint name="joint_big_arm_joint_7" type="revolute">
+  <joint name="big_arm_joint_7" type="revolute">
     <parent link="big_arm_link_6"/>
     <child link="big_arm_link_7"/>
@@ -152,5 +152,5 @@
     <limit lower="-1.5708" upper="1.5708" velocity="100" effort="100"/> <!-- MADE UP NUMBERS JUST FOR TESTING -->
   </joint>
-  <joint name="joint_big_arm_joint_8" type="revolute">
+  <joint name="big_arm_joint_8" type="revolute">
     <parent link="big_arm_link_7"/>
     <child link="big_arm_link_8"/>

File: gateway_description/xacro/little_arm_macro.xacro (robot description, xacro)
@@ -112,15 +112,15 @@
     </collision>
   </link>
-  <joint name="joint_little_arm_joint_0" type="fixed">
+  <joint name="little_arm_joint_0" type="fixed">
     <parent link="${parent}"/>
     <child link="little_arm_link_0"/>
     <xacro:insert_block name="origin"/>
   </joint>
-  <joint name="joint_little_arm_joint_1" type="fixed">
+  <joint name="little_arm_joint_1" type="fixed">
     <parent link="little_arm_link_0"/>
     <child link="little_arm_link_1"/>
     <origin xyz="13.984 -1.3352 -1.3367" rpy="2.3562 0.0 0.0"/>
   </joint>
-  <joint name="joint_little_arm_joint_2" type="revolute">
+  <joint name="little_arm_joint_2" type="revolute">
     <parent link="little_arm_link_1"/>
     <child link="little_arm_link_2"/>
@@ -129,5 +129,5 @@
     <origin xyz="0.44043 0.010424 0.29487" rpy="0.0 0.0 0.0"/>
   </joint>
-  <joint name="joint_little_arm_joint_3" type="revolute">
+  <joint name="little_arm_joint_3" type="revolute">
     <parent link="little_arm_link_2"/>
     <child link="little_arm_link_3"/>
@@ -136,5 +136,5 @@
     <limit lower="-1.5708" upper="1.5708" velocity="100" effort="100"/> <!-- MADE UP NUMBERS JUST FOR TESTING -->
   </joint>
-  <joint name="joint_little_arm_joint_4" type="revolute">
+  <joint name="little_arm_joint_4" type="revolute">
     <parent link="little_arm_link_3"/>
     <child link="little_arm_link_4"/>
@@ -143,5 +143,5 @@
     <limit lower="-1.5708" upper="1.5708" velocity="100" effort="100"/> <!-- MADE UP NUMBERS JUST FOR TESTING -->
   </joint>
-  <joint name="joint_little_arm_joint_5" type="revolute">
+  <joint name="little_arm_joint_5" type="revolute">
     <parent link="little_arm_link_4"/>
     <child link="little_arm_link_5"/>
@@ -150,5 +150,5 @@
     <limit lower="-1.5708" upper="1.5708" velocity="100" effort="100"/> <!-- MADE UP NUMBERS JUST FOR TESTING -->
   </joint>
-  <joint name="joint_little_arm_joint_6" type="revolute">
+  <joint name="little_arm_joint_6" type="revolute">
     <parent link="little_arm_link_5"/>
     <child link="little_arm_link_6"/>
@@ -157,5 +157,5 @@
     <limit lower="-1.5708" upper="1.5708" velocity="100" effort="100"/> <!-- MADE UP NUMBERS JUST FOR TESTING -->
   </joint>
-  <joint name="joint_little_arm_joint_7" type="revolute">
+  <joint name="little_arm_joint_7" type="revolute">
     <parent link="little_arm_link_6"/>
     <child link="little_arm_link_7"/>
@@ -164,5 +164,5 @@
     <limit lower="-1.5708" upper="1.5708" velocity="100" effort="100"/> <!-- MADE UP NUMBERS JUST FOR TESTING -->
   </joint>
-  <joint name="joint_little_arm_joint_8" type="revolute">
+  <joint name="little_arm_joint_8" type="revolute">
     <parent link="little_arm_link_7"/>
     <child link="little_arm_link_8"/>
@@ -171,5 +171,5 @@
     <limit lower="-1.5708" upper="1.5708" velocity="100" effort="100"/> <!-- MADE UP NUMBERS JUST FOR TESTING -->
   </joint>
-  <joint name="joint_little_arm_joint_9" type="revolute">
+  <joint name="little_arm_joint_9" type="revolute">
     <parent link="little_arm_link_8"/>
     <child link="little_arm_link_9"/>
