Commit message: Fix joint axes for little arm

File: gateway_description/xacro/little_arm_macro.xacro (robot description, xacro)
@@ -125,5 +125,5 @@
     <parent link="little_arm_link_1"/>
     <child link="little_arm_link_2"/>
-    <axis xyz="0 0 1"/>
+    <axis xyz="1 0 0"/>
     <limit lower="-1.5708" upper="1.5708" velocity="100" effort="100"/> <!-- MADE UP NUMBERS JUST FOR TESTING -->
     <origin xyz="0.44043 0.010424 0.29487" rpy="0.0 0.0 0.0"/>
@@ -133,5 +133,5 @@
     <child link="little_arm_link_3"/>
     <origin xyz="0.38687 -0.008157 0.011094" rpy="0.0 0.0  0.0"/>
-    <axis xyz="0 1 0"/>
+    <axis xyz="1 0 0"/>
     <limit lower="-1.5708" upper="1.5708" velocity="100" effort="100"/> <!-- MADE UP NUMBERS JUST FOR TESTING -->
   </joint>
@@ -140,5 +140,5 @@
     <child link="little_arm_link_4"/>
     <origin xyz="0.097745 0.0 -0.10467" rpy="0.0 0.0 1.5708"/>
-    <axis xyz="1 0 0"/>
+    <axis xyz="0 0 1"/>
     <limit lower="-1.5708" upper="1.5708" velocity="100" effort="100"/> <!-- MADE UP NUMBERS JUST FOR TESTING -->
   </joint>
@@ -147,5 +147,5 @@
     <child link="little_arm_link_5"/>
     <origin xyz="-0.006176 -0.10467 -0.094197" rpy="0.0 0.0 0.0"/>
-    <axis xyz="1 0 0"/>
+    <axis xyz="0 1 0"/>
     <limit lower="-1.5708" upper="1.5708" velocity="100" effort="100"/> <!-- MADE UP NUMBERS JUST FOR TESTING -->
   </joint>
@@ -154,5 +154,5 @@
     <child link="little_arm_link_6"/>
     <origin xyz="0.47551 -0.21354 0.008568" rpy="0.0 -0.6108 0.0"/>
-    <axis xyz="1 0 0"/>
+    <axis xyz="0 1 0"/>
     <limit lower="-1.5708" upper="1.5708" velocity="100" effort="100"/> <!-- MADE UP NUMBERS JUST FOR TESTING -->
   </joint>
@@ -168,5 +168,5 @@
     <child link="little_arm_link_8"/>
     <origin xyz="0.10062 -0.10467 -0.014366" rpy="0.0 0.0 0.0"/>
-    <axis xyz="0 0 1"/>
+    <axis xyz="1 0 0"/>
     <limit lower="-1.5708" upper="1.5708" velocity="100" effort="100"/> <!-- MADE UP NUMBERS JUST FOR TESTING -->
   </joint>

Commit message: Fix little arm axes

File: gateway_description/xacro/little_arm_macro.xacro (robot description, xacro)
@@ -125,7 +125,7 @@
     <parent link="little_arm_link_1"/>
     <child link="little_arm_link_2"/>
-    <axis xyz="0 0 1"/>
+    <origin xyz="0.44043 0.010424 0.29487" rpy="0.0 0.0 0.0"/>
+    <axis xyz="1 0 0"/>
     <limit lower="-1.5708" upper="1.5708" velocity="3.1416" effort="100"/> <!-- MADE UP NUMBERS JUST FOR TESTING -->
-    <origin xyz="0.44043 0.010424 0.29487" rpy="0.0 0.0 0.0"/>
   </joint>
   <joint name="little_arm_joint_3" type="revolute">
@@ -133,5 +133,5 @@
     <child link="little_arm_link_3"/>
     <origin xyz="0.38687 -0.008157 0.011094" rpy="0.0 0.0  0.0"/>
-    <axis xyz="0 1 0"/>
+    <axis xyz="1 0 0"/>
     <limit lower="-1.5708" upper="1.5708" velocity="3.1416" effort="100"/> <!-- MADE UP NUMBERS JUST FOR TESTING -->
   </joint>
@@ -140,5 +140,5 @@
     <child link="little_arm_link_4"/>
     <origin xyz="0.097745 0.0 -0.10467" rpy="0.0 0.0 1.5708"/>
-    <axis xyz="1 0 0"/>
+    <axis xyz="0 0 1"/>
     <limit lower="-1.5708" upper="1.5708" velocity="3.1416" effort="100"/> <!-- MADE UP NUMBERS JUST FOR TESTING -->
   </joint>
@@ -147,5 +147,5 @@
     <child link="little_arm_link_5"/>
     <origin xyz="-0.006176 -0.10467 -0.094197" rpy="0.0 0.0 0.0"/>
-    <axis xyz="1 0 0"/>
+    <axis xyz="0 1 0"/>
     <limit lower="-1.5708" upper="1.5708" velocity="3.1416" effort="100"/> <!-- MADE UP NUMBERS JUST FOR TESTING -->
   </joint>
@@ -154,5 +154,5 @@
     <child link="little_arm_link_6"/>
     <origin xyz="0.47551 -0.21354 0.008568" rpy="0.0 -0.6108 0.0"/>
-    <axis xyz="1 0 0"/>
+    <axis xyz="0 1 0"/>
     <limit lower="-1.5708" upper="1.5708" velocity="3.1416" effort="100"/> <!-- MADE UP NUMBERS JUST FOR TESTING -->
   </joint>
@@ -168,5 +168,5 @@
     <child link="little_arm_link_8"/>
     <origin xyz="0.10062 -0.10467 -0.014366" rpy="0.0 0.0 0.0"/>
-    <axis xyz="0 0 1"/>
+    <axis xyz="1 0 0"/>
     <limit lower="-1.5708" upper="1.5708" velocity="3.1416" effort="100"/> <!-- MADE UP NUMBERS JUST FOR TESTING -->
   </joint>
