Commit message: increased joint range of both arms -pi -> pi

File: gateway_description/xacro/big_arm_macro.xacro (robot description, xacro)
@@ -114,5 +114,5 @@
     <child link="big_arm_link_2"/>
     <axis xyz="0 0 1"/>
-    <limit lower="-1.5708" upper="1.5708" velocity="100" effort="100"/> <!-- MADE UP NUMBERS JUST FOR TESTING -->
+    <limit lower="-3.14" upper="3.14" velocity="3.1416" effort="100"/> <!-- MADE UP NUMBERS JUST FOR TESTING -->
     <origin xyz="0.0 0.0 0.4409" rpy="0.0 0.0 0.8726648"/>
   </joint>
@@ -122,5 +122,5 @@
     <origin xyz="0.0 -0.177 0.1515" rpy="2.98023e-8 0.0  1.862645e-8"/>
     <axis xyz="0 1 0"/>
-    <limit lower="-1.5708" upper="1.5708" velocity="100" effort="100"/> <!-- MADE UP NUMBERS JUST FOR TESTING -->
+    <limit lower="-3.14" upper="3.14" velocity="3.1416" effort="100"/> <!-- MADE UP NUMBERS JUST FOR TESTING -->
   </joint>
   <joint name="big_arm_joint_4" type="revolute">
@@ -129,5 +129,5 @@
     <origin xyz="0.17432 -0.1594 0.0" rpy="0.95993114 0.0 0.0"/>
     <axis xyz="1 0 0"/>
-    <limit lower="-1.5708" upper="1.5708" velocity="100" effort="100"/> <!-- MADE UP NUMBERS JUST FOR TESTING -->
+    <limit lower="-3.14" upper="3.14" velocity="3.1416" effort="100"/> <!-- MADE UP NUMBERS JUST FOR TESTING -->
   </joint>
   <joint name="big_arm_joint_5" type="revolute">
@@ -136,5 +136,5 @@
     <origin xyz="0.3503 -0.004789 3.6578" rpy="1.3089968 0.0 0.0"/>
     <axis xyz="1 0 0"/>
-    <limit lower="-1.5708" upper="1.5708" velocity="100" effort="100"/> <!-- MADE UP NUMBERS JUST FOR TESTING -->
+    <limit lower="-3.14" upper="3.14" velocity="3.1416" effort="100"/> <!-- MADE UP NUMBERS JUST FOR TESTING -->
   </joint>
   <joint name="big_arm_joint_6" type="revolute">
@@ -143,5 +143,5 @@
     <origin xyz="0.3503 0.004781 -3.6578" rpy="-0.5235989 0.0 0.0"/>
     <axis xyz="1 0 0"/>
-    <limit lower="-1.5708" upper="1.5708" velocity="100" effort="100"/> <!-- MADE UP NUMBERS JUST FOR TESTING -->
+    <limit lower="-3.14" upper="3.14" velocity="3.1416" effort="100"/> <!-- MADE UP NUMBERS JUST FOR TESTING -->
   </joint>
   <joint name="big_arm_joint_7" type="revolute">
@@ -150,5 +150,5 @@
     <origin xyz="0.17429 -0.15194 0.0" rpy="0.0 0.0 0.0"/>
     <axis xyz="0 1 0"/>
-    <limit lower="-1.5708" upper="1.5708" velocity="100" effort="100"/> <!-- MADE UP NUMBERS JUST FOR TESTING -->
+    <limit lower="-3.14" upper="3.14" velocity="3.1416" effort="100"/> <!-- MADE UP NUMBERS JUST FOR TESTING -->
   </joint>
   <joint name="big_arm_joint_8" type="revolute">
@@ -157,5 +157,5 @@
     <origin xyz="-0.004217 -0.1708 -0.181" rpy="0.0 0.0 0.0"/>
     <axis xyz="0 0 1"/>
-    <limit lower="-1.5708" upper="1.5708" velocity="100" effort="100"/> <!-- MADE UP NUMBERS JUST FOR TESTING -->
+    <limit lower="-3.14" upper="3.14" velocity="3.1416" effort="100"/> <!-- MADE UP NUMBERS JUST FOR TESTING -->
   </joint>
   </xacro:macro>

File: gateway_description/xacro/little_arm_macro.xacro (robot description, xacro)
@@ -126,6 +126,5 @@
     <child link="little_arm_link_2"/>
     <axis xyz="1 0 0"/>
-    <limit lower="-1.5708" upper="1.5708" velocity="100" effort="100"/> <!-- MADE UP NUMBERS JUST FOR TESTING -->
-    <origin xyz="0.44043 0.010424 0.29487" rpy="0.0 0.0 0.0"/>
+    <limit lower="-3.14" upper="3.14" velocity="3.1416" effort="100"/> <!-- MADE UP NUMBERS JUST FOR TESTING -->
   </joint>
   <joint name="little_arm_joint_3" type="revolute">
@@ -134,5 +133,5 @@
     <origin xyz="0.38687 -0.008157 0.011094" rpy="0.0 0.0  0.0"/>
     <axis xyz="1 0 0"/>
-    <limit lower="-1.5708" upper="1.5708" velocity="100" effort="100"/> <!-- MADE UP NUMBERS JUST FOR TESTING -->
+    <limit lower="-3.14" upper="3.14" velocity="3.1416" effort="100"/> <!-- MADE UP NUMBERS JUST FOR TESTING -->
   </joint>
   <joint name="little_arm_joint_4" type="revolute">
@@ -141,5 +140,5 @@
     <origin xyz="0.097745 0.0 -0.10467" rpy="0.0 0.0 1.5708"/>
     <axis xyz="0 0 1"/>
-    <limit lower="-1.5708" upper="1.5708" velocity="100" effort="100"/> <!-- MADE UP NUMBERS JUST FOR TESTING -->
+    <limit lower="-3.14" upper="3.14" velocity="3.1416" effort="100"/> <!-- MADE UP NUMBERS JUST FOR TESTING -->
   </joint>
   <joint name="little_arm_joint_5" type="revolute">
@@ -148,5 +147,5 @@
     <origin xyz="-0.006176 -0.10467 -0.094197" rpy="0.0 0.0 0.0"/>
     <axis xyz="0 1 0"/>
-    <limit lower="-1.5708" upper="1.5708" velocity="100" effort="100"/> <!-- MADE UP NUMBERS JUST FOR TESTING -->
+    <limit lower="-3.14" upper="3.14" velocity="3.1416" effort="100"/> <!-- MADE UP NUMBERS JUST FOR TESTING -->
   </joint>
   <joint name="little_arm_joint_6" type="revolute">
@@ -155,5 +154,5 @@
     <origin xyz="0.47551 -0.21354 0.008568" rpy="0.0 -0.6108 0.0"/>
     <axis xyz="0 1 0"/>
-    <limit lower="-1.5708" upper="1.5708" velocity="100" effort="100"/> <!-- MADE UP NUMBERS JUST FOR TESTING -->
+    <limit lower="-3.14" upper="3.14" velocity="3.1416" effort="100"/> <!-- MADE UP NUMBERS JUST FOR TESTING -->
   </joint>
   <joint name="little_arm_joint_7" type="revolute">
@@ -162,5 +161,5 @@
     <origin xyz="0.47551 -0.21354 0.008567" rpy="0.0 0.4363324 0.0"/>
     <axis xyz="0 1 0"/>
-    <limit lower="-1.5708" upper="1.5708" velocity="100" effort="100"/> <!-- MADE UP NUMBERS JUST FOR TESTING -->
+    <limit lower="-3.14" upper="3.14" velocity="3.1416" effort="100"/> <!-- MADE UP NUMBERS JUST FOR TESTING -->
   </joint>
   <joint name="little_arm_joint_8" type="revolute">
@@ -169,5 +168,5 @@
     <origin xyz="0.10062 -0.10467 -0.014366" rpy="0.0 0.0 0.0"/>
     <axis xyz="1 0 0"/>
-    <limit lower="-1.5708" upper="1.5708" velocity="100" effort="100"/> <!-- MADE UP NUMBERS JUST FOR TESTING -->
+    <limit lower="-3.14" upper="3.14" velocity="3.1416" effort="100"/> <!-- MADE UP NUMBERS JUST FOR TESTING -->
   </joint>
   <joint name="little_arm_joint_9" type="revolute">
@@ -176,5 +175,5 @@
     <origin xyz="0.10467 0.000167 -0.10062" rpy="0.0 0.0 0.0"/>
     <axis xyz="0 0 1"/>
-    <limit lower="-1.5708" upper="1.5708" velocity="100" effort="100"/> <!-- MADE UP NUMBERS JUST FOR TESTING -->
+    <limit lower="-3.14" upper="3.14" velocity="3.1416" effort="100"/> <!-- MADE UP NUMBERS JUST FOR TESTING -->
   </joint>
   </xacro:macro>

Commit message: increased joint range of both arms -pi -> pi

File: gateway_description/xacro/big_arm_macro.xacro (robot description, xacro)
@@ -114,5 +114,5 @@
     <child link="big_arm_link_2"/>
     <axis xyz="0 0 1"/>
-    <limit lower="-1.5708" upper="1.5708" velocity="3.1416" effort="100"/> <!-- MADE UP NUMBERS JUST FOR TESTING -->
+    <limit lower="-3.14" upper="3.14" velocity="3.1416" effort="100"/> <!-- MADE UP NUMBERS JUST FOR TESTING -->
     <origin xyz="0.0 0.0 0.4409" rpy="0.0 0.0 0.8726648"/>
   </joint>
@@ -122,5 +122,5 @@
     <origin xyz="0.0 -0.177 0.1515" rpy="2.98023e-8 0.0  1.862645e-8"/>
     <axis xyz="0 1 0"/>
-    <limit lower="-1.5708" upper="1.5708" velocity="3.1416" effort="100"/> <!-- MADE UP NUMBERS JUST FOR TESTING -->
+    <limit lower="-3.14" upper="3.14" velocity="3.1416" effort="100"/> <!-- MADE UP NUMBERS JUST FOR TESTING -->
   </joint>
   <joint name="big_arm_joint_4" type="revolute">
@@ -129,5 +129,5 @@
     <origin xyz="0.17432 -0.1594 0.0" rpy="0.95993114 0.0 0.0"/>
     <axis xyz="1 0 0"/>
-    <limit lower="-1.5708" upper="1.5708" velocity="3.1416" effort="100"/> <!-- MADE UP NUMBERS JUST FOR TESTING -->
+    <limit lower="-3.14" upper="3.14" velocity="3.1416" effort="100"/> <!-- MADE UP NUMBERS JUST FOR TESTING -->
   </joint>
   <joint name="big_arm_joint_5" type="revolute">
@@ -136,5 +136,5 @@
     <origin xyz="0.3503 -0.004789 3.6578" rpy="1.3089968 0.0 0.0"/>
     <axis xyz="1 0 0"/>
-    <limit lower="-1.5708" upper="1.5708" velocity="3.1416" effort="100"/> <!-- MADE UP NUMBERS JUST FOR TESTING -->
+    <limit lower="-3.14" upper="3.14" velocity="3.1416" effort="100"/> <!-- MADE UP NUMBERS JUST FOR TESTING -->
   </joint>
   <joint name="big_arm_joint_6" type="revolute">
@@ -143,5 +143,5 @@
     <origin xyz="0.3503 0.004781 -3.6578" rpy="-0.5235989 0.0 0.0"/>
     <axis xyz="1 0 0"/>
-    <limit lower="-1.5708" upper="1.5708" velocity="3.1416" effort="100"/> <!-- MADE UP NUMBERS JUST FOR TESTING -->
+    <limit lower="-3.14" upper="3.14" velocity="3.1416" effort="100"/> <!-- MADE UP NUMBERS JUST FOR TESTING -->
   </joint>
   <joint name="big_arm_joint_7" type="revolute">
@@ -150,5 +150,5 @@
     <origin xyz="0.17429 -0.15194 0.0" rpy="0.0 0.0 0.0"/>
     <axis xyz="0 1 0"/>
-    <limit lower="-1.5708" upper="1.5708" velocity="3.1416" effort="100"/> <!-- MADE UP NUMBERS JUST FOR TESTING -->
+    <limit lower="-3.14" upper="3.14" velocity="3.1416" effort="100"/> <!-- MADE UP NUMBERS JUST FOR TESTING -->
   </joint>
   <joint name="big_arm_joint_8" type="revolute">
@@ -157,5 +157,5 @@
     <origin xyz="-0.004217 -0.1708 -0.181" rpy="0.0 0.0 0.0"/>
     <axis xyz="0 0 1"/>
-    <limit lower="-1.5708" upper="1.5708" velocity="3.1416" effort="100"/> <!-- MADE UP NUMBERS JUST FOR TESTING -->
+    <limit lower="-3.14" upper="3.14" velocity="3.1416" effort="100"/> <!-- MADE UP NUMBERS JUST FOR TESTING -->
   </joint>
   </xacro:macro>

File: gateway_description/xacro/little_arm_macro.xacro (robot description, xacro)
@@ -127,5 +127,5 @@
     <origin xyz="0.44043 0.010424 0.29487" rpy="0.0 0.0 0.0"/>
     <axis xyz="1 0 0"/>
-    <limit lower="-1.5708" upper="1.5708" velocity="3.1416" effort="100"/> <!-- MADE UP NUMBERS JUST FOR TESTING -->
+    <limit lower="-3.14" upper="3.14" velocity="3.1416" effort="100"/> <!-- MADE UP NUMBERS JUST FOR TESTING -->
   </joint>
   <joint name="little_arm_joint_3" type="revolute">
@@ -134,5 +134,5 @@
     <origin xyz="0.38687 -0.008157 0.011094" rpy="0.0 0.0  0.0"/>
     <axis xyz="1 0 0"/>
-    <limit lower="-1.5708" upper="1.5708" velocity="3.1416" effort="100"/> <!-- MADE UP NUMBERS JUST FOR TESTING -->
+    <limit lower="-3.14" upper="3.14" velocity="3.1416" effort="100"/> <!-- MADE UP NUMBERS JUST FOR TESTING -->
   </joint>
   <joint name="little_arm_joint_4" type="revolute">
@@ -141,5 +141,5 @@
     <origin xyz="0.097745 0.0 -0.10467" rpy="0.0 0.0 1.5708"/>
     <axis xyz="0 0 1"/>
-    <limit lower="-1.5708" upper="1.5708" velocity="3.1416" effort="100"/> <!-- MADE UP NUMBERS JUST FOR TESTING -->
+    <limit lower="-3.14" upper="3.14" velocity="3.1416" effort="100"/> <!-- MADE UP NUMBERS JUST FOR TESTING -->
   </joint>
   <joint name="little_arm_joint_5" type="revolute">
@@ -148,5 +148,5 @@
     <origin xyz="-0.006176 -0.10467 -0.094197" rpy="0.0 0.0 0.0"/>
     <axis xyz="0 1 0"/>
-    <limit lower="-1.5708" upper="1.5708" velocity="3.1416" effort="100"/> <!-- MADE UP NUMBERS JUST FOR TESTING -->
+    <limit lower="-3.14" upper="3.14" velocity="3.1416" effort="100"/> <!-- MADE UP NUMBERS JUST FOR TESTING -->
   </joint>
   <joint name="little_arm_joint_6" type="revolute">
@@ -155,5 +155,5 @@
     <origin xyz="0.47551 -0.21354 0.008568" rpy="0.0 -0.6108 0.0"/>
     <axis xyz="0 1 0"/>
-    <limit lower="-1.5708" upper="1.5708" velocity="3.1416" effort="100"/> <!-- MADE UP NUMBERS JUST FOR TESTING -->
+    <limit lower="-3.14" upper="3.14" velocity="3.1416" effort="100"/> <!-- MADE UP NUMBERS JUST FOR TESTING -->
   </joint>
   <joint name="little_arm_joint_7" type="revolute">
@@ -162,5 +162,5 @@
     <origin xyz="0.47551 -0.21354 0.008567" rpy="0.0 0.4363324 0.0"/>
     <axis xyz="0 1 0"/>
-    <limit lower="-1.5708" upper="1.5708" velocity="3.1416" effort="100"/> <!-- MADE UP NUMBERS JUST FOR TESTING -->
+    <limit lower="-3.14" upper="3.14" velocity="3.1416" effort="100"/> <!-- MADE UP NUMBERS JUST FOR TESTING -->
   </joint>
   <joint name="little_arm_joint_8" type="revolute">
@@ -169,5 +169,5 @@
     <origin xyz="0.10062 -0.10467 -0.014366" rpy="0.0 0.0 0.0"/>
     <axis xyz="1 0 0"/>
-    <limit lower="-1.5708" upper="1.5708" velocity="3.1416" effort="100"/> <!-- MADE UP NUMBERS JUST FOR TESTING -->
+    <limit lower="-3.14" upper="3.14" velocity="3.1416" effort="100"/> <!-- MADE UP NUMBERS JUST FOR TESTING -->
   </joint>
   <joint name="little_arm_joint_9" type="revolute">
@@ -176,5 +176,5 @@
     <origin xyz="0.10467 0.000167 -0.10062" rpy="0.0 0.0 0.0"/>
     <axis xyz="0 0 1"/>
-    <limit lower="-1.5708" upper="1.5708" velocity="3.1416" effort="100"/> <!-- MADE UP NUMBERS JUST FOR TESTING -->
+    <limit lower="-3.14" upper="3.14" velocity="3.1416" effort="100"/> <!-- MADE UP NUMBERS JUST FOR TESTING -->
   </joint>
   </xacro:macro>
