Commit message: Added files to launch gazebo sim of gateway with both arms working

File: robots/little_arm.urdf.xacro (robot description, xacro)
@@ -1,7 +1,11 @@
 <?xml version="1.0"?>
 <robot xmlns:xacro="http://ros.org/wiki/xacro" name="little_arm">
+  <xacro:arg name="parent_link" default="root" />
   <xacro:include filename="$(find gateway_description)/xacro/little_arm_macro.xacro"/>
-  <link name="root"/>
-  <xacro:little_arm parent="root">
+  <!-- Gazebo - ROS2 Control macro -->
+  <xacro:include filename="$(find gateway_description)/xacro/little_arm.gazebo.xacro" />
+  <xacro:gateway_little_arm_gazebo command_interface="position" />
+  <link name="$(arg parent_link)"/>
+  <xacro:little_arm parent="$(arg parent_link)">
     <origin xyz="0.0 0.0 0.0" rpy="0.0 0.4363 -1.396"/>
   </xacro:little_arm>

File: xacro/big_arm_macro.xacro (robot description, xacro)
@@ -2,5 +2,5 @@
 <robot xmlns:xacro="http://ros.org/wiki/xacro" name="big_arm">
   <!-- BIG ARM -->
-  <xacro:macro name="big_arm" params=" parent:='' *origin ">
+  <xacro:macro name="big_arm" params=" parent:='' effort:=2332 velocity:=0.0698 *origin ">
   <link name="big_arm_link_0"/>
   <link name="big_arm_link_1">
@@ -16,7 +16,7 @@
     </collision>
     <inertial>
-      <origin rpy="0 -1.5708 0" xyz="0.25082 0 -0.175"/>
-      <mass value="105.98"/>
-      <inertia ixx="12.19" ixy="0" ixz="0" iyy="12.19" iyz="0" izz="3.061"/>
+      <origin rpy="0 0.0 0" xyz="0.0 0.0 0.0"/>
+      <mass value="199.32"/>
+      <inertia ixx="5.32" ixy="0.08" ixz="0.05" iyy="5.45" iyz="-0.48" izz="3.41"/>
     </inertial>
   </link>
@@ -33,7 +33,7 @@
     </collision>
     <inertial>
-      <origin rpy="0 0 0" xyz="0.175 0 -0.25082"/>
-      <mass value="105.98"/>
-      <inertia ixx="12.19" ixy="0" ixz="0" iyy="12.13" iyz="0" izz="3.061"/>
+      <origin rpy="0 0 0" xyz="0.0003 0.0119 0.1538"/>
+      <mass value="114.07"/>
+      <inertia ixx="1.15" ixy="0" ixz="0" iyy="1.57" iyz="0.07" izz="1.219"/>
     </inertial>
   </link>
@@ -50,7 +50,7 @@
     </collision>
     <inertial>
-      <origin rpy="3.14 0 0" xyz="4.0 0 -0.175"/>
-      <mass value="314.88"/>
-      <inertia ixx="15.41" ixy="0" ixz="0" iyy="2094.71" iyz="0" izz="2103.19"/>
+      <origin rpy="0.0 0.0 0.0" xyz="0.027 -0.158 -0.00389"/>
+      <mass value="104.23"/>
+      <inertia ixx="1.461" ixy="-0.004688" ixz="-0.00272" iyy="1.267" iyz="-0.004355" izz="1.2999"/>
     </inertial>
   </link>
@@ -66,8 +66,8 @@
       </geometry>
     </collision>
-    <inertial>
-      <origin rpy="0 0 0" xyz="-3.6 0 -0.175"/>
-      <mass value="279.2"/>
-      <inertia ixx="9.522" ixy="0" ixz="0" iyy="1966.28" iyz="0" izz="1966.28"/>
+    <inertial auto="true">
+      <origin rpy="0 0 0" xyz="0.068 -0.0215 2.311"/>
+      <mass value="1009.8049"/>
+      <inertia ixx="1039.65" ixy="-4.50" ixz="75.17" iyy="1063.62" iyz="5.92" izz="38.36"/>
     </inertial>
   </link>
@@ -84,7 +84,7 @@
     </collision>
     <inertial>
-      <origin rpy="1.5708 0 0" xyz="0 0 0.0"/>
-      <mass value="105.98"/>
-      <inertia ixx="8.305" ixy="0" ixz="0" iyy="3.061" iyz="0" izz="8.0386"/>
+      <origin rpy="0 0 0" xyz="0.27 0.0052 -1.6147"/>
+      <mass value="1105.62"/>
+      <inertia ixx="1630.99" ixy="-4.146" ixz="-75.05" iyy="1657.002" iyz="-5.089" izz="40.19"/>
     </inertial>
   </link>
@@ -101,7 +101,7 @@
     </collision>
     <inertial>
-      <origin rpy="0 -1.5708 0" xyz="0 0 0"/>
-      <mass value="105.98"/>
-      <inertia ixx="12.13" ixy="0" ixz="0" iyy="12.13" iyz="0" izz="3.061"/>
+      <origin rpy="0 0 0" xyz="0.1549 -0.017 -0.00327"/>
+      <mass value="96.32"/>
+      <inertia ixx="1.11" ixy="0.0299" ixz="0.0082" iyy="1.333" iyz="0.0096" izz="1.1131"/>
     </inertial>
   </link>
@@ -118,7 +118,7 @@
     </collision>
     <inertial>
-      <origin rpy="0 1.5708 0" xyz="0 0 -0.5"/>
-      <mass value="243.66"/>
-      <inertia ixx="9.336" ixy="0" ixz="0" iyy="44.41" iyz="0" izz="44.41"/>
+      <origin rpy="0 0 0" xyz="-0.0289 -0.1639 -0.01698"/>
+      <mass value="123.193"/>
+      <inertia ixx="1.7418" ixy="-0.0206" ixz="-0.000706" iyy="1.72372" iyz="-0.07149" izz="1.7646"/>
     </inertial>
   </link>
@@ -135,7 +135,7 @@
     </collision>
     <inertial>
-      <origin rpy="0 1.5708 0" xyz="0 0 -0.5"/>
-      <mass value="243.66"/>
-      <inertia ixx="9.336" ixy="0" ixz="0" iyy="44.41" iyz="0" izz="44.41"/>
+      <origin rpy="0 0 0" xyz="0.001862 0.00626 -0.2257"/>
+      <mass value="199.327"/>
+      <inertia ixx="4.778" ixy="-0.068" ixz="0.0139" iyy="4.571" iyz="0.0458" izz="3.311"/>
     </inertial>
   </link>
@@ -154,5 +154,5 @@
     <child link="big_arm_link_2"/>
     <axis xyz="0 0 1"/>
-    <limit lower="-3.14" upper="3.14" velocity="3.1416" effort="100"/> <!-- MADE UP NUMBERS JUST FOR TESTING -->
+    <limit lower="-3.14" upper="3.14" velocity="${velocity}" effort="${effort}"/>
     <origin xyz="0.0 0.0 0.4409" rpy="0.0 0.0 0.8726648"/>
   </joint>
@@ -162,5 +162,5 @@
     <origin xyz="0.0 -0.177 0.1515" rpy="2.98023e-8 0.0  1.862645e-8"/>
     <axis xyz="0 1 0"/>
-    <limit lower="-3.14" upper="3.14" velocity="3.1416" effort="100"/> <!-- MADE UP NUMBERS JUST FOR TESTING -->
+    <limit lower="-3.14" upper="3.14" velocity="${velocity}" effort="${effort}"/>
   </joint>
   <joint name="big_arm_joint_4" type="revolute">
@@ -169,5 +169,5 @@
     <origin xyz="0.17432 -0.1594 0.0" rpy="0.95993114 0.0 0.0"/>
     <axis xyz="1 0 0"/>
-    <limit lower="-3.14" upper="3.14" velocity="3.1416" effort="100"/> <!-- MADE UP NUMBERS JUST FOR TESTING -->
+    <limit lower="-3.14" upper="3.14" velocity="${velocity}" effort="${effort}"/>
   </joint>
   <joint name="big_arm_joint_5" type="revolute">
@@ -176,5 +176,5 @@
     <origin xyz="0.3503 -0.004789 3.6578" rpy="1.3089968 0.0 0.0"/>
     <axis xyz="1 0 0"/>
-    <limit lower="-3.14" upper="3.14" velocity="3.1416" effort="100"/> <!-- MADE UP NUMBERS JUST FOR TESTING -->
+    <limit lower="-3.14" upper="3.14" velocity="${velocity}" effort="${effort}"/>
   </joint>
   <joint name="big_arm_joint_6" type="revolute">
@@ -183,5 +183,5 @@
     <origin xyz="0.3503 0.004781 -3.6578" rpy="-0.5235989 0.0 0.0"/>
     <axis xyz="1 0 0"/>
-    <limit lower="-3.14" upper="3.14" velocity="3.1416" effort="100"/> <!-- MADE UP NUMBERS JUST FOR TESTING -->
+    <limit lower="-3.14" upper="3.14" velocity="${velocity}" effort="${effort}"/>
   </joint>
   <joint name="big_arm_joint_7" type="revolute">
@@ -190,5 +190,5 @@
     <origin xyz="0.17429 -0.15194 0.0" rpy="0.0 0.0 0.0"/>
     <axis xyz="0 1 0"/>
-    <limit lower="-3.14" upper="3.14" velocity="3.1416" effort="100"/> <!-- MADE UP NUMBERS JUST FOR TESTING -->
+    <limit lower="-3.14" upper="3.14" velocity="${velocity}" effort="${effort}"/>
   </joint>
   <joint name="big_arm_joint_8" type="revolute">
@@ -197,5 +197,5 @@
     <origin xyz="-0.004217 -0.1708 -0.181" rpy="0.0 0.0 0.0"/>
     <axis xyz="0 0 1"/>
-    <limit lower="-3.14" upper="3.14" velocity="3.1416" effort="100"/> <!-- MADE UP NUMBERS JUST FOR TESTING -->
+    <limit lower="-3.14" upper="3.14" velocity="${velocity}" effort="${effort}"/>
   </joint>
   </xacro:macro>

File: xacro/little_arm.gazebo.xacro (robot description, xacro)
@@ -1,10 +1,10 @@
 <?xml version="1.0" ?>
 <robot xmlns:xacro="http://wiki.ros.org/xacro">
-  <xacro:macro name="gateway_big_arm_gazebo" params="command_interface:=position">
+  <xacro:macro name="gateway_little_arm_gazebo" params="command_interface:=position">
   <ros2_control name="GazeboSystem" type="system">
       <hardware>
           <plugin>gz_ros2_control/GazeboSimSystem</plugin>
       </hardware>
-      <joint name="big_arm_joint_2">
+      <joint name="little_arm_joint_2">
           <command_interface name="${command_interface}"/>
           <state_interface name="position"/>
@@ -12,5 +12,5 @@
           <state_interface name="effort"/>
       </joint>
-      <joint name="big_arm_joint_3">
+      <joint name="little_arm_joint_3">
           <command_interface name="${command_interface}"/>
           <state_interface name="position"/>
@@ -18,5 +18,5 @@
           <state_interface name="effort"/>
       </joint>
-      <joint name="big_arm_joint_4">
+      <joint name="little_arm_joint_4">
           <command_interface name="${command_interface}"/>
           <state_interface name="position"/>
@@ -24,5 +24,5 @@
           <state_interface name="effort"/>
       </joint>
-      <joint name="big_arm_joint_5">
+      <joint name="little_arm_joint_5">
           <command_interface name="${command_interface}"/>
           <state_interface name="position"/>
@@ -30,5 +30,5 @@
           <state_interface name="effort"/>
       </joint>
-      <joint name="big_arm_joint_6">
+      <joint name="little_arm_joint_6">
           <command_interface name="${command_interface}"/>
           <state_interface name="position"/>
@@ -36,5 +36,5 @@
           <state_interface name="effort"/>
       </joint>
-      <joint name="big_arm_joint_7">
+      <joint name="little_arm_joint_7">
           <command_interface name="${command_interface}"/>
           <state_interface name="position"/>
@@ -42,5 +42,11 @@
           <state_interface name="effort"/>
       </joint>
-      <joint name="big_arm_joint_8">
+      <joint name="little_arm_joint_8">
+          <command_interface name="${command_interface}"/>
+          <state_interface name="position"/>
+          <state_interface name="velocity"/>
+          <state_interface name="effort"/>
+      </joint>
+      <joint name="little_arm_joint_9">
           <command_interface name="${command_interface}"/>
           <state_interface name="position"/>
@@ -51,8 +57,8 @@
   <gazebo>
       <plugin filename="gz_ros2_control-system" name="gz_ros2_control::GazeboSimROS2ControlPlugin">
-        <parameters>$(find gateway_description)/config/big_arm_control.yaml</parameters>
+        <parameters>$(find gateway_description)/config/little_arm_control.yaml</parameters>
         <ros>
-          <namespace>big_arm</namespace>
-          <remapping>/robot_description:=/big_arm/robot_description</remapping>
+          <namespace>little_arm</namespace>
+          <remapping>/robot_description:=/little_arm/robot_description</remapping>
         </ros>
       </plugin>

File: xacro/little_arm_macro.xacro (robot description, xacro)
@@ -2,5 +2,5 @@
 <robot xmlns:xacro="http://ros.org/wiki/xacro" name="little_arm">
   <!-- LITTLE ARM -->
-  <xacro:macro name="little_arm" params=" parent:='' *origin ">
+  <xacro:macro name="little_arm" params=" parent:='' effort:=2332 velocity:=0.0698 *origin ">
   <link name="little_arm_link_0"/>
   <link name="little_arm_link_1">
@@ -15,4 +15,9 @@
       </geometry>
     </collision>
+    <inertial>
+      <origin rpy="0 0.0 0" xyz="0.0 0.0 0.0"/>
+      <mass value="550.422"/>
+      <inertia ixx="24.6499" ixy="-0.291088" ixz="-0.102784" iyy="23.824" iyz="-4.06098" izz="23.7613"/>
+    </inertial>
   </link>
   <link name="little_arm_link_2">
@@ -27,4 +32,9 @@
       </geometry>
     </collision>
+    <inertial>
+      <origin rpy="0 0.0 0" xyz="0.173508 -0.0300499 -0.0499662"/>
+      <mass value="33.5272"/>
+      <inertia ixx="0.580764" ixy="-0.0770547" ixz="-0.0476339" iyy="0.497335" iyz="-0.0269257" izz="0.446148"/>
+    </inertial>
   </link>
   <link name="little_arm_link_3">
@@ -39,4 +49,9 @@
       </geometry>
     </collision>
+    <inertial>
+      <origin rpy="0 0.0 0" xyz="0.104632 -6.30748e-06 0.0133201"/>
+      <mass value="33.7845"/>
+      <inertia ixx="0.157109" ixy="3.37505e-06" ixz="0.00253518" iyy="0.14345" iyz="4.38914e-05" izz="0.222663"/>
+    </inertial>
   </link>
   <link name="little_arm_link_4">
@@ -51,4 +66,9 @@
       </geometry>
     </collision>
+    <inertial>
+      <origin rpy="0 0.0 0" xyz="-0.00622422 0.0129621 -0.104538"/>
+      <mass value="33.8161"/>
+      <inertia ixx="0.147648" ixy="-0.00351409" ixz="0.000100141" iyy="0.221961" iyz="-0.0042235" izz="0.160461"/>
+    </inertial>
   </link>
   <link name="little_arm_link_5">
@@ -63,4 +83,9 @@
       </geometry>
     </collision>
+    <inertial>
+      <origin rpy="0 0.0 0" xyz="0.250363 -0.0718547 0.00510753"/>
+      <mass value="102.114"/>
+      <inertia ixx="0.724753" ixy="0.526541" ixz="-0.000815258" iyy="4.80145" iyz="-7.6685e-05" izz="4.84377"/>
+    </inertial>
   </link>
   <link name="little_arm_link_6">
@@ -75,4 +100,9 @@
       </geometry>
     </collision>
+    <inertial>
+      <origin rpy="0 0.0 0" xyz="0.231175 -0.0909595 -0.000464751"/>
+      <mass value="100.374"/>
+      <inertia ixx="0.805978" ixy="0.444523" ixz="-0.0704152" iyy="4.7502" iyz="-0.0217411" izz="4.89759"/>
+    </inertial>
   </link>
   <link name="little_arm_link_7">
@@ -87,4 +117,9 @@
       </geometry>
     </collision>
+    <inertial>
+      <origin rpy="0 0.0 0" xyz="-0.00201876 -0.0987844 -0.012305"/>
+      <mass value="35.5519"/>
+      <inertia ixx="0.226425" ixy="-0.00140961" ixz="0.00011871" iyy="0.242722" iyz="-0.00272485" izz="0.207642"/>
+    </inertial>
   </link>
   <link name="little_arm_link_8">
@@ -99,4 +134,9 @@
       </geometry>
     </collision>
+    <inertial>
+      <origin rpy="0 0.0 0" xyz="0.101053 -0.00153106 0.0255484"/>
+      <mass value="35.4028"/>
+      <inertia ixx="0.181332" ixy="0.000209396" ixz="-0.00521308" iyy="0.148371" iyz="-0.000702566" izz="0.216962"/>
+    </inertial>
   </link>
   <link name="little_arm_link_9">
@@ -111,4 +151,9 @@
       </geometry>
     </collision>
+    <inertial>
+      <origin rpy="0.0 0.0 0.0" xyz="0.0345403 -0.0115104 -0.202042"/>
+      <mass value="77.6497"/>
+      <inertia ixx="1.02124" ixy="0.0555304" ixz="0.0666044" iyy="1.10279" iyz="-0.0188412" izz="0.645531"/>
+    </inertial>
   </link>
   <joint name="little_arm_joint_0" type="fixed">
@@ -127,5 +172,5 @@
     <origin xyz="0.44043 0.010424 0.29487" rpy="0.0 0.0 0.0"/>
     <axis xyz="1 0 0"/>
-    <limit lower="-3.14" upper="3.14" velocity="3.1416" effort="100"/> <!-- MADE UP NUMBERS JUST FOR TESTING -->
+    <limit lower="-3.14" upper="3.14" velocity="${velocity}" effort="${effort}"/>
   </joint>
   <joint name="little_arm_joint_3" type="revolute">
@@ -134,5 +179,5 @@
     <origin xyz="0.38687 -0.008157 0.011094" rpy="0.0 0.0  0.0"/>
     <axis xyz="1 0 0"/>
-    <limit lower="-3.14" upper="3.14" velocity="3.1416" effort="100"/> <!-- MADE UP NUMBERS JUST FOR TESTING -->
+    <limit lower="-3.14" upper="3.14" velocity="${velocity}" effort="${effort}"/>
   </joint>
   <joint name="little_arm_joint_4" type="revolute">
@@ -141,5 +186,5 @@
     <origin xyz="0.097745 0.0 -0.10467" rpy="0.0 0.0 1.5708"/>
     <axis xyz="0 0 1"/>
-    <limit lower="-3.14" upper="3.14" velocity="3.1416" effort="100"/> <!-- MADE UP NUMBERS JUST FOR TESTING -->
+    <limit lower="-3.14" upper="3.14" velocity="${velocity}" effort="${effort}"/>
   </joint>
   <joint name="little_arm_joint_5" type="revolute">
@@ -148,5 +193,5 @@
     <origin xyz="-0.006176 -0.10467 -0.094197" rpy="0.0 0.0 0.0"/>
     <axis xyz="0 1 0"/>
-    <limit lower="-3.14" upper="3.14" velocity="3.1416" effort="100"/> <!-- MADE UP NUMBERS JUST FOR TESTING -->
+    <limit lower="-3.14" upper="3.14" velocity="${velocity}" effort="${effort}"/>
   </joint>
   <joint name="little_arm_joint_6" type="revolute">
@@ -155,5 +200,5 @@
     <origin xyz="0.47551 -0.21354 0.008568" rpy="0.0 -0.6108 0.0"/>
     <axis xyz="0 1 0"/>
-    <limit lower="-3.14" upper="3.14" velocity="3.1416" effort="100"/> <!-- MADE UP NUMBERS JUST FOR TESTING -->
+    <limit lower="-3.14" upper="3.14" velocity="${velocity}" effort="${effort}"/>
   </joint>
   <joint name="little_arm_joint_7" type="revolute">
@@ -162,5 +207,5 @@
     <origin xyz="0.47551 -0.21354 0.008567" rpy="0.0 0.4363324 0.0"/>
     <axis xyz="0 1 0"/>
-    <limit lower="-3.14" upper="3.14" velocity="3.1416" effort="100"/> <!-- MADE UP NUMBERS JUST FOR TESTING -->
+    <limit lower="-3.14" upper="3.14" velocity="${velocity}" effort="${effort}"/>
   </joint>
   <joint name="little_arm_joint_8" type="revolute">
@@ -169,5 +214,5 @@
     <origin xyz="0.10062 -0.10467 -0.014366" rpy="0.0 0.0 0.0"/>
     <axis xyz="1 0 0"/>
-    <limit lower="-3.14" upper="3.14" velocity="3.1416" effort="100"/> <!-- MADE UP NUMBERS JUST FOR TESTING -->
+    <limit lower="-3.14" upper="3.14" velocity="${velocity}" effort="${effort}"/>
   </joint>
   <joint name="little_arm_joint_9" type="revolute">
@@ -176,5 +221,5 @@
     <origin xyz="0.10467 0.000167 -0.10062" rpy="0.0 0.0 0.0"/>
     <axis xyz="0 0 1"/>
-    <limit lower="-3.14" upper="3.14" velocity="3.1416" effort="100"/> <!-- MADE UP NUMBERS JUST FOR TESTING -->
+    <limit lower="-3.14" upper="3.14" velocity="${velocity}" effort="${effort}"/>
   </joint>
   </xacro:macro>
