Commit message: Big arm moves in Gazebo, with moon on the horizon and gateway base. Arm is a bit swingy

File: robots/big_arm.urdf.xacro (robot description, xacro)
@@ -1,7 +1,11 @@
 <?xml version="1.0"?>
 <robot xmlns:xacro="http://ros.org/wiki/xacro" name="big_arm">
+  <xacro:arg name="parent_link" default="root" />
   <xacro:include filename="$(find gateway_description)/xacro/big_arm_macro.xacro"/>
-  <link name="root"/>
-  <xacro:big_arm parent="root">
+  <!-- Gazebo - ROS2 Control macro -->
+  <xacro:include filename="$(find gateway_description)/xacro/big_arm.gazebo.xacro" />
+  <xacro:gateway_big_arm_gazebo command_interface="position" />
+  <link name="$(arg parent_link)"/>
+  <xacro:big_arm parent="$(arg parent_link)">
     <origin xyz="0.0 0.0 0.0" rpy="0.0 0.4363 -1.396"/>
   </xacro:big_arm>

File: xacro/big_arm_macro.xacro (robot description, xacro)
@@ -15,4 +15,9 @@
       </geometry>
     </collision>
+    <inertial>
+      <origin rpy="0 -1.5708 0" xyz="0.25082 0 -0.175"/>
+      <mass value="105.98"/>
+      <inertia ixx="12.19" ixy="0" ixz="0" iyy="12.19" iyz="0" izz="3.061"/>
+    </inertial>
   </link>
   <link name="big_arm_link_2">
@@ -27,4 +32,9 @@
       </geometry>
     </collision>
+    <inertial>
+      <origin rpy="0 0 0" xyz="0.175 0 -0.25082"/>
+      <mass value="105.98"/>
+      <inertia ixx="12.19" ixy="0" ixz="0" iyy="12.13" iyz="0" izz="3.061"/>
+    </inertial>
   </link>
   <link name="big_arm_link_3">
@@ -39,4 +49,9 @@
       </geometry>
     </collision>
+    <inertial>
+      <origin rpy="3.14 0 0" xyz="4.0 0 -0.175"/>
+      <mass value="314.88"/>
+      <inertia ixx="15.41" ixy="0" ixz="0" iyy="2094.71" iyz="0" izz="2103.19"/>
+    </inertial>
   </link>
   <link name="big_arm_link_4">
@@ -51,4 +66,9 @@
       </geometry>
     </collision>
+    <inertial>
+      <origin rpy="0 0 0" xyz="-3.6 0 -0.175"/>
+      <mass value="279.2"/>
+      <inertia ixx="9.522" ixy="0" ixz="0" iyy="1966.28" iyz="0" izz="1966.28"/>
+    </inertial>
   </link>
   <link name="big_arm_link_5">
@@ -63,4 +83,9 @@
       </geometry>
     </collision>
+    <inertial>
+      <origin rpy="1.5708 0 0" xyz="0 0 0.0"/>
+      <mass value="105.98"/>
+      <inertia ixx="8.305" ixy="0" ixz="0" iyy="3.061" iyz="0" izz="8.0386"/>
+    </inertial>
   </link>
   <link name="big_arm_link_6">
@@ -75,4 +100,9 @@
       </geometry>
     </collision>
+    <inertial>
+      <origin rpy="0 -1.5708 0" xyz="0 0 0"/>
+      <mass value="105.98"/>
+      <inertia ixx="12.13" ixy="0" ixz="0" iyy="12.13" iyz="0" izz="3.061"/>
+    </inertial>
   </link>
   <link name="big_arm_link_7">
@@ -87,4 +117,9 @@
       </geometry>
     </collision>
+    <inertial>
+      <origin rpy="0 1.5708 0" xyz="0 0 -0.5"/>
+      <mass value="243.66"/>
+      <inertia ixx="9.336" ixy="0" ixz="0" iyy="44.41" iyz="0" izz="44.41"/>
+    </inertial>
   </link>
   <link name="big_arm_link_8">
@@ -99,4 +134,9 @@
       </geometry>
     </collision>
+    <inertial>
+      <origin rpy="0 1.5708 0" xyz="0 0 -0.5"/>
+      <mass value="243.66"/>
+      <inertia ixx="9.336" ixy="0" ixz="0" iyy="44.41" iyz="0" izz="44.41"/>
+    </inertial>
   </link>
   <joint name="big_arm_joint_0" type="fixed">

File: xacro/gateway_body_macro.xacro (robot description, xacro)
@@ -19,4 +19,9 @@
       </geometry>
     </collision>
+    <inertial>
+      <origin rpy="0 1.5708 0" xyz="0 0 -0.5"/>
+      <mass value="243.66"/>
+      <inertia ixx="9.336" ixy="0" ixz="0" iyy="44.41" iyz="0" izz="44.41"/>
+    </inertial>
   </link>
   <link name="ihab">
@@ -31,4 +36,9 @@
       </geometry>
     </collision>
+    <inertial>
+      <origin rpy="0 1.5708 0" xyz="0 0 -0.5"/>
+      <mass value="243.66"/>
+      <inertia ixx="9.336" ixy="0" ixz="0" iyy="44.41" iyz="0" izz="44.41"/>
+    </inertial>
   </link>
   <link name="ng_halo">
@@ -43,4 +53,9 @@
       </geometry>
     </collision>
+    <inertial>
+      <origin rpy="0 1.5708 0" xyz="0 0 -0.5"/>
+      <mass value="243.66"/>
+      <inertia ixx="9.336" ixy="0" ixz="0" iyy="44.41" iyz="0" izz="44.41"/>
+    </inertial>
   </link>
   <link name="ermxl">
@@ -55,4 +70,9 @@
       </geometry>
     </collision>
+    <inertial>
+      <origin rpy="0 1.5708 0" xyz="0 0 -0.5"/>
+      <mass value="243.66"/>
+      <inertia ixx="9.336" ixy="0" ixz="0" iyy="44.41" iyz="0" izz="44.41"/>
+    </inertial>
   </link>
   <link name="maxar_ppe">
@@ -67,4 +87,9 @@
       </geometry>
     </collision>
+    <inertial>
+      <origin rpy="0 1.5708 0" xyz="0 0 -0.5"/>
+      <mass value="243.66"/>
+      <inertia ixx="9.336" ixy="0" ixz="0" iyy="44.41" iyz="0" izz="44.41"/>
+    </inertial>
   </link>
 <!--  <joint name="joint_root_mover" type="fixed">

Commit message: Added a camera because why not

File: robots/big_arm.urdf.xacro (robot description, xacro)
@@ -14,5 +14,30 @@
     <parent link="big_arm_link_8"/>
     <child link="big_arm_link_tcp"/>
-    <origin xyz="0 0 0" rpy="0 0 0"/>
+    <origin xyz="0 0 -0.50" rpy="0 1.5708 1.5708"/>
   </joint>
+    <gazebo reference="big_arm_link_tcp">
+      <sensor type="camera" name="camera_sensor">
+          <visualize>1</visualize>
+          <update_rate>10.0</update_rate>
+          <camera>
+              <pose>1.0 0 0 0 0 -1.57</pose>
+              <horizontal_fov>1.3962634</horizontal_fov>
+              <image>
+                  <width>800</width>
+                  <height>800</height>
+                  <format>R8G8B8</format>
+              </image>
+              <clip>
+              <near>0.01</near>
+              <far>100</far>
+              </clip>
+              <noise>
+              <type>gaussian</type>
+              <stddev>0.007</stddev>
+              </noise>
+          </camera>
+          <always_on>1</always_on>
+          <topic>image_raw</topic>
+      </sensor>
+  </gazebo>
 </robot>

Commit message: Moved camera gazebo stuff within the gazebo macro file to be easily found

File: robots/big_arm.urdf.xacro (robot description, xacro)
@@ -14,30 +14,5 @@
     <parent link="big_arm_link_8"/>
     <child link="big_arm_link_tcp"/>
-    <origin xyz="0 0 -0.50" rpy="0 1.5708 1.5708"/>
+    <origin xyz="0 0 0" rpy="0 0 0"/>
   </joint>
-    <gazebo reference="big_arm_link_tcp">
-      <sensor type="camera" name="camera_sensor">
-          <visualize>1</visualize>
-          <update_rate>10.0</update_rate>
-          <camera>
-              <pose>1.0 0 0 0 0 -1.57</pose>
-              <horizontal_fov>1.3962634</horizontal_fov>
-              <image>
-                  <width>800</width>
-                  <height>800</height>
-                  <format>R8G8B8</format>
-              </image>
-              <clip>
-              <near>0.01</near>
-              <far>100</far>
-              </clip>
-              <noise>
-              <type>gaussian</type>
-              <stddev>0.007</stddev>
-              </noise>
-          </camera>
-          <always_on>1</always_on>
-          <topic>image_raw</topic>
-      </sensor>
-  </gazebo>
 </robot>

File: xacro/big_arm.gazebo.xacro (robot description, xacro)
@@ -58,4 +58,36 @@
       </plugin>
   </gazebo>
+  <!-- Simulate camera at the end of big arm-->
+  <link name="big_arm_dummy_camera_link"/>
+  <joint name="big_arm_camera_joint" type="fixed">
+    <parent link="big_arm_link_8"/>
+    <child link="big_arm_dummy_camera_link"/>
+    <origin xyz="0 0 -0.50" rpy="0 1.5708 1.5708"/>
+  </joint>
+  <gazebo reference="big_arm_dummy_camera_link">
+      <sensor type="camera" name="camera_sensor">
+          <visualize>1</visualize>
+          <update_rate>10.0</update_rate>
+          <camera>
+              <pose>1.0 0 0 0 0 -1.57</pose>
+              <horizontal_fov>1.3962634</horizontal_fov>
+              <image>
+                  <width>800</width>
+                  <height>800</height>
+                  <format>R8G8B8</format>
+              </image>
+              <clip>
+              <near>0.01</near>
+              <far>100</far>
+              </clip>
+              <noise>
+              <type>gaussian</type>
+              <stddev>0.007</stddev>
+              </noise>
+          </camera>
+          <always_on>1</always_on>
+          <topic>image_raw</topic>
+      </sensor>
+  </gazebo>
   </xacro:macro>
 </robot>
